Commit message: Add separate end effector link to sequential robot

File: tests/sequential_planar_arm.urdf (robot description, URDF)
Before this commit: robot simple, 5 links, 4 joints
Links:
- added link link3; visual box size=0.4 0.2 0.2
- link eef: geometry visual box size=0.15 0.2 0.2
Joints:
- added joint l2_to_l3: type revolute, parent link2, child link3, origin xyz=0.6 0.0 0.0, axis 0 0 1, limit lower=-1.0 upper=1.0 effort=1000.0 velocity=0.5
- joint ee: axis 0 0 1 -> (none); limit lower=-1.0 upper=1.0 effort=1000.0 velocity=0.5 -> (none); origin xyz=0.6 0.0 0.0 -> xyz=0.3 0.0 0.0; parent link2 -> link3; type revolute -> fixed
