Commit message: Getting joint limits of whole chain
Added methods to grab the velocity and effort limits
of all joints in a chain at once. Updated tests
accordingly.

File: tests/joint_no_limit_robot.urdf (robot description, URDF)
Before this commit: robot joint_limit_robot, 6 links, 5 joints
Joints:
- joint joint1: limit lower=9 upper=10 effort=5 velocity=1 -> effort=5 velocity=1
- joint joint2: limit lower=10 upper=11 effort=6 velocity=2 -> effort=6 velocity=2
- joint joint3: limit lower=11 upper=12 effort=7 velocity=3 -> effort=7 velocity=3
- joint joint4: limit lower=12 upper=13 effort=8 velocity=4 -> effort=8 velocity=4
